File: binary_in_7seg.sch (KiCad schematic (older format))
At the start: 15 parts

Commit message: Starting layout
Parts:
- P1: renamed from P?; footprint (none) -> Housings_DIP:DIP-14_W7.62mm
- Q1, Q2: renamed from Q?; footprint (none) -> TO_SOT_Packages_SMD:SOT-323
- R1, R10, R2, R3, R4, R5, R6, R7, R8, R9: renamed from R?; footprint (none) -> Resistors_SMD:R_0402
- S1: renamed from S?; footprint (none) -> Displays_7-Segment:7SEGMENT-LED__HDSM531_HDSM533_SMD
- U1: renamed from U?; footprint (none) -> Housings_SSOP:TSSOP-16_4.4x5mm_Pitch0.65mm
Changed lines of the file:
@@
 $EndDescr
 $Comp
-L 7SEGM S?
+L 7SEGM S1
 U 1 1 57DA1C00
 P 9050 3200
-F 0 "S?" H 9050 3850 50  0000 C CNN
+F 0 "S1" H 9050 3850 50  0000 C CNN
 F 1 "7SEGM" H 9050 2550 50  0000 C CNN
-F 2 "" H 9050 3200 50  0000 C CNN
+F 2 "Displays_7-Segment:7SEGMENT-LED__HDSM531_HDSM533_SMD" H 9050 3200 50  0001 C CNN
 F 3 "" H 9050 3200 50  0000 C CNN
 	1    9050 3200
@@
 $EndComp
 $Comp
-L CD4543 U?
+L CD4543 U1
 U 1 1 57DEBCF8
 P 6650 3100
-F 0 "U?" H 6800 3700 60  0000 C CNN
+F 0 "U1" H 6800 3700 60  0000 C CNN
 F 1 "CD4543" H 6450 3700 60  0000 C CNN
-F 2 "" H 6650 3100 60  0000 C CNN
+F 2 "Housings_SSOP:TSSOP-16_4.4x5mm_Pitch0.65mm" H 6650 3100 60  0001 C CNN
 F 3 "" H 6650 3100 60  0000 C CNN
 	1    6650 3100
@@
 $EndComp
 $Comp
-L R R?
+L R R3
 U 1 1 57DEBD77
 P 7500 2900
-F 0 "R?" V 7580 2900 50  0000 C CNN
+F 0 "R3" V 7580 2900 50  0000 C CNN
 F 1 "R" V 7500 2900 50  0000 C CNN
-F 2 "" V 7430 2900 50  0000 C CNN
+F 2 "Resistors_SMD:R_0402" V 7430 2900 50  0001 C CNN
 F 3 "" H 7500 2900 50  0000 C CNN
 	1    7500 2900
@@
 $EndComp
 $Comp
-L R R?
+L R R7
 U 1 1 57DEBDAF
 P 7800 3000
-F 0 "R?" V 7880 3000 50  0000 C CNN
+F 0 "R7" V 7880 3000 50  0000 C CNN
 F 1 "R" V 7800 3000 50  0000 C CNN
-F 2 "" V 7730 3000 50  0000 C CNN
+F 2 "Resistors_SMD:R_0402" V 7730 3000 50  0001 C CNN
 F 3 "" H 7800 3000 50  0000 C CNN
 	1    7800 3000
@@
 $EndComp
 $Comp
-L R R?
+L R R4
 U 1 1 57DEBDD4
 P 7500 3100
-F 0 "R?" V 7580 3100 50  0000 C CNN
+F 0 "R4" V 7580 3100 50  0000 C CNN
 F 1 "R" V 7500 3100 50  0000 C CNN
-F 2 "" V 7430 3100 50  0000 C CNN
+F 2 "Resistors_SMD:R_0402" V 7430 3100 50  0001 C CNN
 F 3 "" H 7500 3100 50  0000 C CNN
 	1    7500 3100
@@
 $EndComp
 $Comp
-L R R?
+L R R8
 U 1 1 57DEBDFA
 P 7800 3200
-F 0 "R?" V 7880 3200 50  0000 C CNN
+F 0 "R8" V 7880 3200 50  0000 C CNN
 F 1 "R" V 7800 3200 50  0000 C CNN
-F 2 "" V 7730 3200 50  0000 C CNN
+F 2 "Resistors_SMD:R_0402" V 7730 3200 50  0001 C CNN
 F 3 "" H 7800 3200 50  0000 C CNN
 	1    7800 3200
@@
 $EndComp
 $Comp
-L R R?
+L R R5
 U 1 1 57DEBE38
 P 7500 3300
-F 0 "R?" V 7580 3300 50  0000 C CNN
+F 0 "R5" V 7580 3300 50  0000 C CNN
 F 1 "R" V 7500 3300 50  0000 C CNN
-F 2 "" V 7430 3300 50  0000 C CNN
+F 2 "Resistors_SMD:R_0402" V 7430 3300 50  0001 C CNN
 F 3 "" H 7500 3300 50  0000 C CNN
 	1    7500 3300
@@
 $EndComp
 $Comp
-L R R?
+L R R9
 U 1 1 57DEBE84
 P 7800 3400
-F 0 "R?" V 7880 3400 50  0000 C CNN
+F 0 "R9" V 7880 3400 50  0000 C CNN
 F 1 "R" V 7800 3400 50  0000 C CNN
-F 2 "" V 7730 3400 50  0000 C CNN
+F 2 "Resistors_SMD:R_0402" V 7730 3400 50  0001 C CNN
 F 3 "" H 7800 3400 50  0000 C CNN
 	1    7800 3400
@@
 $EndComp
 $Comp
-L R R?
+L R R6
 U 1 1 57DEBEB6
 P 7500 3500
-F 0 "R?" V 7580 3500 50  0000 C CNN
+F 0 "R6" V 7580 3500 50  0000 C CNN
 F 1 "R" V 7500 3500 50  0000 C CNN
-F 2 "" V 7430 3500 50  0000 C CNN
+F 2 "Resistors_SMD:R_0402" V 7430 3500 50  0001 C CNN
 F 3 "" H 7500 3500 50  0000 C CNN
 	1    7500 3500
@@
 	7650 2900 8300 2900
 $Comp
-L DIL14 P?
+L DIL14 P1
 U 1 1 57E00234
 P 3950 3000
-F 0 "P?" H 3950 3400 50  0000 C CNN
+F 0 "P1" H 3950 3400 50  0000 C CNN
 F 1 "DIL14" V 3950 3000 50  0000 C CNN
-F 2 "" H 3950 3000 50  0000 C CNN
+F 2 "Housings_DIP:DIP-14_W7.62mm" H 3950 3000 50  0001 C CNN
 F 3 "" H 3950 3000 50  0000 C CNN
 	1    3950 3000
@@
 $EndComp
 $Comp
-L GND #PWR?
+L GND #PWR01
 U 1 1 57E00275
 P 3500 3400
-F 0 "#PWR?" H 3500 3150 50  0001 C CNN
+F 0 "#PWR01" H 3500 3150 50  0001 C CNN
 F 1 "GND" H 3500 3250 50  0000 C CNN
 F 2 "" H 3500 3400 50  0000 C CNN
@@
 	3500 3300 3600 3300
 $Comp
-L VDD #PWR?
+L VDD #PWR02
 U 1 1 57E00343
 P 4450 2600
-F 0 "#PWR?" H 4450 2450 50  0001 C CNN
+F 0 "#PWR02" H 4450 2450 50  0001 C CNN
 F 1 "VDD" H 4450 2750 50  0000 C CNN
 F 2 "" H 4450 2600 50  0000 C CNN
@@
 	4450 2700 4450 2600
 Wire Wire Line
-	4300 3300 5700 3300
-Wire Wire Line
-	5700 3300 5700 3300
-Wire Wire Line
-	5700 3300 6050 3300
+	4300 3300 6050 3300
 $Bitmap
 Pos 2150 4350
@@
 	3150 2900 3600 2900
 $Comp
-L +5V #PWR?
+L +5V #PWR03
 U 1 1 57E00A6F
 P 3450 2600
-F 0 "#PWR?" H 3450 2450 50  0001 C CNN
+F 0 "#PWR03" H 3450 2450 50  0001 C CNN
 F 1 "+5V" H 3450 2740 50  0000 C CNN
 F 2 "" H 3450 2600 50  0000 C CNN
@@
 	3450 2700 3600 2700
 $Comp
-L +5V #PWR?
+L +5V #PWR04
 U 1 1 57E00AF1
 P 8200 2650
-F 0 "#PWR?" H 8200 2500 50  0001 C CNN
+F 0 "#PWR04" H 8200 2500 50  0001 C CNN
 F 1 "+5V" H 8200 2790 50  0000 C CNN
 F 2 "" H 8200 2650 50  0000 C CNN
@@
 $EndComp
 Wire Wire Line
-	8200 2650 8200 2800
-Wire Wire Line
-	8200 2800 8200 3700
+	8200 2650 8200 3700
 Wire Wire Line
 	8200 2800 8300 2800
@@
 	5800 3200 6050 3200
 $Comp
-L GND #PWR?
+L GND #PWR05
 U 1 1 57E00D02
 P 5950 3600
-F 0 "#PWR?" H 5950 3350 50  0001 C CNN
+F 0 "#PWR05" H 5950 3350 50  0001 C CNN
 F 1 "GND" H 5950 3450 50  0000 C CNN
 F 2 "" H 5950 3600 50  0000 C CNN
@@
 $EndComp
 Wire Wire Line
-	5950 3400 5950 3500
-Wire Wire Line
-	5950 3500 5950 3600
+	5950 3400 5950 3600
 Wire Wire Line
 	5950 3500 6050 3500
 $Comp
-L VDD #PWR?
+L VDD #PWR06
 U 1 1 57E00D6F
 P 7350 2600
-F 0 "#PWR?" H 7350 2450 50  0001 C CNN
+F 0 "#PWR06" H 7350 2450 50  0001 C CNN
 F 1 "VDD" H 7350 2750 50  0000 C CNN
 F 2 "" H 7350 2600 50  0000 C CNN
@@
 Connection ~ 5950 3500
 $Comp
-L Q_NMOS_DGS Q?
+L Q_NMOS_DGS Q1
 U 1 1 57E026D3
 P 6800 4000
-F 0 "Q?" H 7100 4050 50  0000 R CNN
+F 0 "Q1" H 7100 4050 50  0000 R CNN
 F 1 "Q_NMOS_DGS" H 7450 3950 50  0000 R CNN
-F 2 "" H 7000 4100 50  0000 C CNN
+F 2 "TO_SOT_Packages_SMD:SOT-323" H 7000 4100 50  0001 C CNN
 F 3 "" H 6800 4000 50  0000 C CNN
 	1    6800 4000
@@
 $EndComp
 $Comp
-L Q_NMOS_DGS Q?
+L Q_NMOS_DGS Q2
 U 1 1 57E0271C
 P 7450 5000
-F 0 "Q?" H 7750 5050 50  0000 R CNN
+F 0 "Q2" H 7750 5050 50  0000 R CNN
 F 1 "Q_NMOS_DGS" H 8100 4950 50  0000 R CNN
-F 2 "" H 7650 5100 50  0000 C CNN
+F 2 "TO_SOT_Packages_SMD:SOT-323" H 7650 5100 50  0001 C CNN
 F 3 "" H 7450 5000 50  0000 C CNN
 	1    7450 5000
@@
 $EndComp
 $Comp
-L GND #PWR?
+L GND #PWR07
 U 1 1 57E027E1
 P 6900 4600
-F 0 "#PWR?" H 6900 4350 50  0001 C CNN
+F 0 "#PWR07" H 6900 4350 50  0001 C CNN
 F 1 "GND" H 6900 4450 50  0000 C CNN
 F 2 "" H 6900 4600 50  0000 C CNN
@@
 $EndComp
 $Comp
-L GND #PWR?
+L GND #PWR08
 U 1 1 57E0284C
 P 7550 5600
-F 0 "#PWR?" H 7550 5350 50  0001 C CNN
+F 0 "#PWR08" H 7550 5350 50  0001 C CNN
 F 1 "GND" H 7550 5450 50  0000 C CNN
 F 2 "" H 7550 5600 50  0000 C CNN
@@
 $EndComp
 Wire Wire Line
-	7550 5200 7550 5500
-Wire Wire Line
-	7550 5500 7550 5600
+	7550 5200 7550 5600
 Wire Wire Line
-	6900 4200 6900 4500
-Wire Wire Line
-	6900 4500 6900 4600
+	6900 4200 6900 4600
 $Comp
-L R R?
+L R R1
 U 1 1 57E02906
 P 6500 4250
-F 0 "R?" V 6580 4250 50  0000 C CNN
+F 0 "R1" V 6580 4250 50  0000 C CNN
 F 1 "R" V 6500 4250 50  0000 C CNN
-F 2 "" V 6430 4250 50  0000 C CNN
+F 2 "Resistors_SMD:R_0402" V 6430 4250 50  0001 C CNN
 F 3 "" H 6500 4250 50  0000 C CNN
 	1    6500 4250
@@
 $EndComp
 $Comp
-L R R?
+L R R2
 U 1 1 57E02947
 P 7150 5250
-F 0 "R?" V 7230 5250 50  0000 C CNN
+F 0 "R2" V 7230 5250 50  0000 C CNN
 F 1 "R" V 7150 5250 50  0000 C CNN
-F 2 "" V 7080 5250 50  0000 C CNN
+F 2 "Resistors_SMD:R_0402" V 7080 5250 50  0001 C CNN
 F 3 "" H 7150 5250 50  0000 C CNN
 	1    7150 5250
@@
 	6500 4100 6500 4000
 Wire Wire Line
-	5600 4000 6500 4000
-Wire Wire Line
-	6500 4000 6600 4000
+	5600 4000 6600 4000
 Wire Wire Line
 	7150 5100 7150 5000
 Wire Wire Line
-	3150 5000 7150 5000
-Wire Wire Line
-	7150 5000 7250 5000
+	3150 5000 7250 5000
 Wire Wire Line
 	7150 5400 7150 5500
@@
 	7550 4800 7550 3700
 Wire Wire Line
-	6900 3700 7550 3700
-Wire Wire Line
-	7550 3700 7650 3700
+	6900 3700 7650 3700
 Wire Wire Line
 	6900 3700 6900 3800
@@
 Connection ~ 7150 5000
 $Comp
-L R R?
+L R R10
 U 1 1 57E0311F
 P 7800 3700
-F 0 "R?" V 7880 3700 50  0000 C CNN
+F 0 "R10" V 7880 3700 50  0000 C CNN
 F 1 "R" V 7800 3700 50  0000 C CNN
-F 2 "" V 7730 3700 50  0000 C CNN
+F 2 "Resistors_SMD:R_0402" V 7730 3700 50  0001 C CNN
 F 3 "" H 7800 3700 50  0000 C CNN
 	1    7800 3700
